File: hw/sch_pcb/UST1BATTD01A.kicad_pcb (KiCad board)
At the start: 2 copper layers, 90.9 x 50.3 mm, 13 parts, among them J1 SM03B-GHS-TB, J2 SM03B-GHS-TB, J3 SM03B-GHS-TB, J4 SM03B-GHS-TB, M1 HOLE, M2 HOLE, M3 HOLE, M4 HOLE

Commit message: Edit PCB
Connections:
- M1 pad 1: GND -> unconnected-(M1-Pad1)
- M2 pad 1: GND -> unconnected-(M2-Pad1)
- M3 pad 1: GND -> unconnected-(M3-Pad1)
- M4 pad 1: GND -> unconnected-(M4-Pad1)
Routing:
- net Net-(D1-Pad1): track 0.00 -> 63.6 mm, vias 0 -> 3
- net Net-(BT1-Pad1): track 0.00 -> 20.3 mm
- net Net-(D2-Pad2): track 0.00 -> 4.99 mm
- net Net-(D1-Pad2): track 0.00 -> 4.98 mm
- added copper zone on B.Cu, net GND
- added copper zone on F.Cu, net GND
Other:
- board text added: "JACHO 2022"
- board text added: "UST.CZ UST1BATTD01A"
- board text removed: "3V6"
- board text removed: "GND"
- board text removed: "OUT"
- board text removed: "UST.CZ USTSIPM01A"
